File: circuit.brd (EAGLE design)
At the start: 50 x 93.8 mm, 18 parts, among them IC1 74HC595N

Commit message: final?
Parts:
- added U$5: SLIDE_SWITCH, HyTechDevices:SLIDE_SWITCH
- U$4: value LED_5MM_RGB -> LED_5MM_RGBSTRAIGHT; device HyTechDevices:LED_5MM_RGB -> HyTechDevices:LED-RGB-THRU
- moved U$2 25.2 mm to (41.1, 24.4), turned to 90 degrees
- moved JP3 15.3 mm to (40.6, 10.2)
- moved JP2 11.5 mm to (24.1, 10.2)
- moved U$4 0.25 mm to (28.2, 82.0), turned to 180 degrees
- renumbered S1 to S3, S2 to S4
Connections:
- new net N$2: U$2.14, U$5.P$2
- net BLUE: now also U$4.4; no longer U$4.1
- net GND: now also U$4.2; no longer U$4.3
- net GREEN: now also U$4.3; no longer U$4.2
- net RED: now also U$4.1; no longer U$4.4
- net VIN: now also U$5.P$3; no longer U$2.14
Routing:
- net GND: track 0.00 -> 62.4 mm, vias 0 -> 2
- net N$8: track 108.4 -> 70.2 mm, vias 9 -> 3
- net N$2: track 0.00 -> 36.8 mm
- net N$6: track 15.4 -> 50.9 mm
- net N$5: track 44.4 -> 55.4 mm
- net VIN: track 75.0 -> 85.7 mm
- net SDA: track 33.9 -> 23.7 mm, vias 1 -> 0
- net REC: track 48.6 -> 56.6 mm, vias 0 -> 1
- net PWM1: track 111.1 -> 104.6 mm
- net BLUE: track 119.7 -> 124.5 mm
- net +3V3: track 206.6 -> 211.4 mm
- net UNFREEZE: track 37.0 -> 40.9 mm, vias 0 -> 1
- net GREEN: track 118.4 -> 120.6 mm
- net RED: track 130.0 -> 129.4 mm
Other:
- board text added: "off"
- board text added: "on"

Commit message: final
Parts:
- U$4: value LED_5MM_RGBSTRAIGHT -> LED_5MM_RGB; device HyTechDevices:LED-RGB-THRU -> HyTechDevices:LED_5MM_RGB
- turned U$4 to 0 degrees
Routing:
- net GREEN: track 120.6 -> 126.8 mm
- net BLUE: track 124.5 -> 126.3 mm
- net RED: track 129.4 -> 130.3 mm
- net SCL: track 24.4 -> 23.7 mm
Changed lines of the file:
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@@
 <param name="rvMicroViaOuter" value="0.25"/>
 <param name="rvMicroViaInner" value="0.25"/>
-<param name="rlMinPadTop" value="0mil"/>
+<param name="rlMinPadTop" value="10mil"/>
 <param name="rlMaxPadTop" value="20mil"/>
-<param name="rlMinPadInner" value="0mil"/>
+<param name="rlMinPadInner" value="10mil"/>
 <param name="rlMaxPadInner" value="20mil"/>
-<param name="rlMinPadBottom" value="0mil"/>
+<param name="rlMinPadBottom" value="10mil"/>
 <param name="rlMaxPadBottom" value="20mil"/>
 <param name="rlMinViaOuter" value="8mil"/>
@@
 <element name="U$1" library="HyTechDevices" package="TEENSY_3.5_SIMPLE" value="TEENSY_3.5" x="2.54" y="29.21" smashed="yes"/>
 <element name="U$2" library="HyTechDevices" package="VGA-15" value="VGA-15" x="41.148" y="24.384" smashed="yes" rot="R90"/>
-<element name="U$4" library="HyTechDevices" package="LED-RGB-THRU" value="LED_5MM_RGBSTRAIGHT" x="28.194" y="82.042" smashed="yes" rot="R180"/>
 <element name="U$5" library="HyTechDevices" package="SLIDE_SWITCH" value="SLIDE_SWITCH" x="28.194" y="21.59" smashed="yes" rot="R180"/>
 <element name="S3" library="switch-omron" package="B3F-40XX" package3d_urn="urn:adsk.eagle:package:27483/1" value="" x="40.64" y="10.16" smashed="yes" rot="R270">
@@
 <attribute name="VALUE" x="19.05" y="13.335" size="1.27" layer="27" ratio="10" rot="R270"/>
 </element>
+<element name="U$4" library="HyTechDevices" package="LED_5MM_RGB" value="LED_5MM_RGB" x="28.194" y="82.042" smashed="yes"/>
 </elements>
 <signals>
@@
 </polygon>
 <contactref element="U$2" pad="1"/>
-<contactref element="U$4" pad="2"/>
 <via x="41.402" y="30.734" extent="1-16" drill="0.5"/>
 <wire x1="41.402" y1="30.734" x2="44.196" y2="27.94" width="0.4064" layer="1"/>
@@
 <wire x1="13.97" y1="49.53" x2="15.24" y2="48.26" width="0.6096" layer="16"/>
 <wire x1="3.81" y1="88.9" x2="3.81" y2="90.17" width="0.8128" layer="16"/>
-<wire x1="3.81" y1="88.9" x2="3.81" y2="87.7474" width="0.8128" layer="16"/>
 <wire x1="3.81" y1="88.9" x2="5.08" y2="88.9" width="0.8128" layer="16"/>
 <wire x1="3.81" y1="88.9" x2="2.54" y2="88.9" width="0.8128" layer="16"/>
@@
 <wire x1="31.75" y1="45.212" x2="31.75" y2="46.99" width="0.8128" layer="16"/>
 <wire x1="31.75" y1="45.212" x2="31.75" y2="44.45" width="0.8128" layer="16"/>
+<contactref element="U$4" pad="2"/>
+<wire x1="3.81" y1="88.9" x2="3.81" y2="87.884" width="0.8128" layer="16"/>
 </signal>
 <signal name="VIN">
@@
 <wire x1="27.94" y1="88.9" x2="27.94" y2="87.63" width="0.6096" layer="16"/>
 <wire x1="27.94" y1="87.63" x2="26.67" y2="86.36" width="0.6096" layer="16"/>
-<wire x1="22.86" y1="86.36" x2="21.59" y2="85.09" width="0.6096" layer="16"/>
+<wire x1="24.13" y1="86.36" x2="21.59" y2="83.82" width="0.6096" layer="16"/>
 <wire x1="21.59" y1="72.39" x2="20.32" y2="71.12" width="0.6096" layer="16"/>
 <wire x1="20.32" y1="71.12" x2="19.05" y2="71.12" width="0.6096" layer="16"/>
-<wire x1="26.67" y1="86.36" x2="22.86" y2="86.36" width="0.6096" layer="16"/>
-<wire x1="21.59" y1="85.09" x2="21.59" y2="72.39" width="0.6096" layer="16"/>
+<wire x1="26.67" y1="86.36" x2="24.13" y2="86.36" width="0.6096" layer="16"/>
+<wire x1="21.59" y1="83.82" x2="21.59" y2="72.39" width="0.6096" layer="16"/>
 </signal>
 <signal name="SDA">
@@
 <wire x1="25.530925" y1="24.13" x2="26.292925" y2="24.892" width="0.6096" layer="16"/>
 <wire x1="26.292925" y1="24.892" x2="29.21" y2="24.892" width="0.6096" layer="16"/>
-<contactref element="U$4" pad="1"/>
-<wire x1="23.876" y1="79.629" x2="26.289" y2="82.042" width="0.6096" layer="16"/>
-<wire x1="23.876" y1="72.644" x2="23.876" y2="79.629" width="0.6096" layer="16"/>
 <wire x1="48.514" y1="50.546" x2="48.514" y2="48.514" width="0.6096" layer="1"/>
 <wire x1="48.514" y1="48.514" x2="48.26" y2="48.26" width="0.6096" layer="1"/>
@@
 <wire x1="34.159" y1="62.361" x2="23.876" y2="72.644" width="0.6096" layer="16"/>
 <wire x1="34.1452" y1="56.7868" x2="34.1452" y2="60.47440625" width="0.6096" layer="16"/>
+<contactref element="U$4" pad="1"/>
+<wire x1="23.876" y1="80.8514" x2="26.035" y2="83.0104" width="0.6096" layer="16"/>
+<wire x1="23.876" y1="72.644" x2="23.876" y2="80.8514" width="0.6096" layer="16"/>
 </signal>
 <signal name="GREEN">
@@
 <wire x1="28.702" y1="27.686" x2="30.988" y2="25.4" width="0.6096" layer="1"/>
 <wire x1="30.988" y1="25.4" x2="35.306" y2="25.4" width="0.6096" layer="1"/>
-<contactref element="U$4" pad="3"/>
-<wire x1="28.8163" y1="80.94970625" x2="28.8163" y2="82.0293" width="0.6096" layer="1"/>
-<wire x1="28.8163" y1="82.0293" x2="28.829" y2="82.042" width="0.6096" layer="1"/>
-<wire x1="23.368" y1="70.612" x2="23.368" y2="75.50140625" width="0.6096" layer="1"/>
-<wire x1="23.368" y1="75.50140625" x2="28.8163" y2="80.94970625" width="0.6096" layer="1"/>
+<wire x1="23.368" y1="70.612" x2="23.368" y2="74.93" width="0.6096" layer="1"/>
+<wire x1="23.368" y1="74.93" x2="23.368" y2="75.50140625" width="0.6096" layer="1"/>
 <wire x1="47.4325375" y1="45.2774625" x2="46.99" y2="45.72" width="0.6096" layer="16"/>
 <wire x1="46.99" y1="45.72" x2="46.99" y2="46.99" width="0.6096" layer="16"/>
@@
 <wire x1="46.99" y1="46.99" x2="46.99" y2="50.669075" width="0.6096" layer="1"/>
 <wire x1="46.99" y1="50.669075" x2="42.261675" y2="55.3974" width="0.6096" layer="1"/>
+<contactref element="U$4" pad="3"/>
+<wire x1="23.368" y1="75.50140625" x2="23.368" y2="83.058" width="0.6096" layer="1"/>
+<wire x1="27.0034" y1="85.09" x2="29.083" y2="83.0104" width="0.6096" layer="1"/>
+<wire x1="23.368" y1="83.058" x2="25.4" y2="85.09" width="0.6096" layer="1"/>
+<wire x1="25.4" y1="85.09" x2="27.0034" y2="85.09" width="0.6096" layer="1"/>
 </signal>
 <signal name="BLUE">
@@
 <wire x1="29.21" y1="30.48" x2="29.21" y2="26.67" width="0.6096" layer="16"/>
 <wire x1="26.67" y1="26.67" x2="26.67" y2="30.48" width="0.6096" layer="16"/>
-<contactref element="U$4" pad="4"/>
 <wire x1="22.606" y1="82.296" x2="25.4" y2="85.09" width="0.6096" layer="16"/>
-<wire x1="30.0863" y1="83.38829375" x2="30.0863" y2="82.0547" width="0.6096" layer="16"/>
-<wire x1="30.0863" y1="82.0547" x2="30.099" y2="82.042" width="0.6096" layer="16"/>
-<wire x1="25.4" y1="85.09" x2="28.38459375" y2="85.09" width="0.6096" layer="16"/>
-<wire x1="28.38459375" y1="85.09" x2="30.0863" y2="83.38829375" width="0.6096" layer="16"/>
+<wire x1="25.4" y1="85.09" x2="27.94" y2="85.09" width="0.6096" layer="16"/>
+<wire x1="27.94" y1="85.09" x2="28.38459375" y2="85.09" width="0.6096" layer="16"/>
 <wire x1="22.606" y1="72.005075" x2="22.606" y2="82.296" width="0.6096" layer="16"/>
-<wire x1="35.306" y1="51.054" x2="35.306" y2="50.8" width="0.6096" layer="16"/>
-<wire x1="35.306" y1="50.8" x2="35.306" y2="42.926" width="0.6096" layer="16"/>
+<wire x1="35.306" y1="51.562" x2="35.306" y2="42.926" width="0.6096" layer="16"/>
 <wire x1="35.306" y1="42.926" x2="34.29" y2="41.91" width="0.6096" layer="16"/>
 <wire x1="34.29" y1="41.91" x2="34.29" y2="26.67" width="0.6096" layer="16"/>
@@
 <wire x1="24.638" y1="59.69" x2="25.908" y2="59.69" width="0.6096" layer="16"/>
 <wire x1="23.622" y1="58.674" x2="24.638" y2="59.69" width="0.6096" layer="16"/>
-<wire x1="35.306" y1="51.054" x2="35.306" y2="51.562" width="0.6096" layer="16"/>
 <wire x1="35.306" y1="51.562" x2="31.7246" y2="55.1434" width="0.6096" layer="16"/>
 <wire x1="31.7246" y1="55.1434" x2="25.1206" y2="55.1434" width="0.6096" layer="16"/>
+<contactref element="U$4" pad="4"/>
+<wire x1="28.38459375" y1="85.09" x2="29.21" y2="85.09" width="0.6096" layer="16"/>
+<wire x1="30.607" y1="83.693" x2="30.607" y2="81.3276" width="0.6096" layer="16"/>
+<wire x1="30.607" y1="81.3276" x2="30.353" y2="81.0736" width="0.6096" layer="16"/>
+<wire x1="29.21" y1="85.09" x2="30.607" y2="83.693" width="0.6096" layer="16"/>
 </signal>
 <signal name="N$5">
